Commit message: Commit del launch

File: robotRangers__autonomousNavigation_puzzleBot/urdf/puzzlebot_jetson_ed_urdf.urdf (robot description, URDF)
Before this commit: robot Puzzlebot Jetson-Lidar Ed., 4 links, 3 joints
Joints:
- joint lw_joint: origin xyz=0.055 0.19 0.0046 -> xyz=0.05 0.087 0.0046
- joint rw_joint: origin xyz=0.055 -0.087 0.0046 -> xyz=0.05 -0.087 0.0046

Commit message: Modificación del URDF

File: robotRangers__autonomousNavigation_puzzleBot/urdf/puzzlebot_jetson_ed_urdf.urdf (robot description, URDF)
Before this commit: robot Puzzlebot Jetson-Lidar Ed., 4 links, 3 joints
Joints:
- joint lw_joint: axis (none) -> 0 1 0; limit (none) -> lower=-3.1416 upper=3.1416 effort=100 velocity=3.14; type continuous -> revolute
- joint rw_joint: axis (none) -> 0 1 0; limit (none) -> lower=-3.1416 upper=3.1416 effort=100 velocity=3.14; type continuous -> revolute
